File: HW/ESP_LT8900.kicad_pcb (KiCad board)
At the start: 2 copper layers, 50 x 50 mm, 38 parts, among them P1 PWR, P2 TTL, P3 I2C, P4 485_EN, P5 RS485, SW1 Reset, SW2 Flash, U1 ESP-07, U2 LT8900, U3 MC78M05CDT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

Commit message: HW &SW Folder Update
Parts:
- added U6: nRF24L01_12x18mm, NRF24L01_12x18mm, B.Cu at (106.5, 140.5)
- U2: footprint BK_Common:LT8900_2.54mmPitch_20x20 -> LT8900_2.54mmPitch_SMD_20x20
- moved ? 19.9 mm to (128.0, 134.6)
- moved ? 16.1 mm to (139.5, 135.1)
Routing:
- net /CSN: track 41.7 -> 54.2 mm, vias 0 -> 1
- net /MISO: track 15.3 -> 27.5 mm, vias 0 -> 1
- net +3V3: track 116.9 -> 126.1 mm, vias 4 -> 6
- net /PKT: track 19.6 -> 26.7 mm, vias 0 -> 1
- net /MOSI: track 16.0 -> 23.0 mm, vias 1 -> 2
- net GND: track 92.0 -> 98.4 mm, vias 4 -> 5
- net /SCK: track 22.2 -> 27.3 mm, vias 0 -> 1
Other:
- board text added: "LT8900"
- board text added: "NRF24L01"
- board text added: "https://github.com/bklemencz/ESP_LT8900"
